Commit message: april_tag & multi robot added

File: grid_robot/urdf/grid_robot.urdf (robot description, URDF)
Before this commit: robot grid_robot, 3 links, 2 joints
Links:
- added link april_tag_link, mass 0.0001; visual box size=0.05 0.05 0.001
- link base_link: mass 0.085712 -> None
Joints:
- added joint april_tag_joint: type fixed, parent base_link, child april_tag_link, origin xyz=0 0 0.013 rpy=0 0 0, axis 0 0 0
