File: grid_hardware/micromouse_eagle/ESpdesign_1.brd (EAGLE design)
At the start: 89.8 x 61 mm, 8 parts

Commit message: new brd added
Parts:
- moved S2 107.1 mm to (45.0, 55.5), flipped to the bottom, turned to 180 degrees
- moved S1 80.9 mm to (46.1, 15.1), turned to 180 degrees
- moved SV4 70.0 mm to (45.8, 43.2), flipped to the bottom, turned to 90 degrees
- moved SV3 61.0 mm to (4.83, 49.7), flipped to the bottom
- moved SV2 56.4 mm to (1.65, 31.0), turned to 270 degrees
- moved SV1 53.9 mm to (1.65, 23.4), turned to 270 degrees
- moved U$1 53.7 mm to (24.4, 28.1), turned to 180 degrees
- moved JP1 32.0 mm to (4.83, 57.7), flipped to the bottom, turned to 270 degrees
Routing:
- net N$41: track 179.2 -> 0.00 mm
- net N$1: track 363.0 -> 302.0 mm
- net P+: track 0.00 -> 47.7 mm
- net 5V: track 0.00 -> 44.6 mm
- net B-: track 0.00 -> 24.5 mm
- net N$40: track 24.4 -> 0.00 mm
- net N$31: track 26.5 -> 2.10 mm
- net N$6: track 25.5 -> 1.50 mm
- net GND: track 0.00 -> 22.5 mm
- net D8: track 0.00 -> 18.6 mm
- net D3: track 0.00 -> 16.5 mm
- net D2: track 0.00 -> 14.6 mm
- net D1: track 0.00 -> 14.6 mm
- net D4: track 0.00 -> 13.9 mm
- net D5: track 0.00 -> 9.97 mm
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