File: grid_hardware/micromouse_eagle/bots_123/ESpdesign.brd (EAGLE design)
At the start: 89.8 x 61 mm, 8 parts

Commit message: added brd pdf
Routing:
- net N$4: track 0.00 -> 302.5 mm
Changed lines of the file:
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@@
 <grid distance="50" unitdist="mil" unit="mil" style="lines" multiple="1" display="no" altdistance="5" altunitdist="mil" altunit="mil"/>
 <layers>
-<layer number="1" name="Top" color="4" fill="1" visible="yes" active="yes"/>
+<layer number="1" name="Top" color="4" fill="1" visible="no" active="yes"/>
 <layer number="16" name="Bottom" color="1" fill="1" visible="yes" active="yes"/>
 <layer number="17" name="Pads" color="2" fill="1" visible="yes" active="yes"/>
 <layer number="18" name="Vias" color="2" fill="1" visible="yes" active="yes"/>
-<layer number="19" name="Unrouted" color="6" fill="1" visible="yes" active="yes"/>
-<layer number="20" name="Dimension" color="24" fill="1" visible="yes" active="yes"/>
-<layer number="21" name="tPlace" color="7" fill="1" visible="yes" active="yes"/>
-<layer number="22" name="bPlace" color="7" fill="1" visible="yes" active="yes"/>
-<layer number="23" name="tOrigins" color="15" fill="1" visible="yes" active="yes"/>
-<layer number="24" name="bOrigins" color="15" fill="1" visible="yes" active="yes"/>
-<layer number="25" name="tNames" color="7" fill="1" visible="yes" active="yes"/>
-<layer number="26" name="bNames" color="7" fill="1" visible="yes" active="yes"/>
-<layer number="27" name="tValues" color="7" fill="1" visible="yes" active="yes"/>
-<layer number="28" name="bValues" color="7" fill="1" visible="yes" active="yes"/>
+<layer number="19" name="Unrouted" color="6" fill="1" visible="no" active="yes"/>
+<layer number="20" name="Dimension" color="24" fill="1" visible="no" active="yes"/>
+<layer number="21" name="tPlace" color="7" fill="1" visible="no" active="yes"/>
+<layer number="22" name="bPlace" color="7" fill="1" visible="no" active="yes"/>
+<layer number="23" name="tOrigins" color="15" fill="1" visible="no" active="yes"/>
+<layer number="24" name="bOrigins" color="15" fill="1" visible="no" active="yes"/>
+<layer number="25" name="tNames" color="7" fill="1" visible="no" active="yes"/>
+<layer number="26" name="bNames" color="7" fill="1" visible="no" active="yes"/>
+<layer number="27" name="tValues" color="7" fill="1" visible="no" active="yes"/>
+<layer number="28" name="bValues" color="7" fill="1" visible="no" active="yes"/>
 <layer number="29" name="tStop" color="7" fill="3" visible="no" active="yes"/>
 <layer number="30" name="bStop" color="7" fill="6" visible="no" active="yes"/>
@@
 <layer number="49" name="Reference" color="7" fill="1" visible="yes" active="yes"/>
 <layer number="50" name="dxf" color="7" fill="1" visible="no" active="no"/>
-<layer number="51" name="tDocu" color="7" fill="1" visible="yes" active="yes"/>
-<layer number="52" name="bDocu" color="7" fill="1" visible="yes" active="yes"/>
+<layer number="51" name="tDocu" color="7" fill="1" visible="no" active="yes"/>
+<layer number="52" name="bDocu" color="7" fill="1" visible="no" active="yes"/>
 <layer number="53" name="tGND_GNDA" color="7" fill="9" visible="no" active="no"/>
 <layer number="54" name="bGND_GNDA" color="1" fill="9" visible="no" active="no"/>
@@
 <text x="17.78" y="44.45" size="1.778" layer="16">CYBORG</text>
 <text x="14.478" y="4.953" size="1.778" layer="16">MADE BY- NIPEN</text>
+<circle x="87.503" y="42.545" radius="1.27" width="0.1524" layer="16"/>
+<circle x="87.503" y="18.288" radius="1.250803125" width="0.1524" layer="16"/>
+<circle x="51.943" y="22.987" radius="1.486496875" width="0.1524" layer="16"/>
+<circle x="51.943" y="37.973" radius="1.419903125" width="0.1524" layer="16"/>
+<circle x="17.018" y="24.765" radius="1.53454375" width="0.1524" layer="16"/>
+<circle x="32.004" y="24.765" radius="1.481059375" width="0.1524" layer="16"/>
+<circle x="32.004" y="36.195" radius="1.52928125" width="0.1524" layer="16"/>
+<circle x="17.018" y="36.195" radius="1.52928125" width="0.1524" layer="16"/>
 </plain>
 <attributes>
@@
 <wire x1="40.25" y1="3.99" x2="40.25" y2="62.09" width="0.001" layer="1"/>
 </signal>
+<signal name="N$4">
+<wire x1="-0.381" y1="60.96" x2="89.916" y2="60.96" width="0.1524" layer="16"/>
+<wire x1="89.916" y1="60.96" x2="89.916" y2="0" width="0.1524" layer="16"/>
+<wire x1="89.916" y1="0" x2="-0.381" y2="0" width="0.1524" layer="16"/>
+<wire x1="-0.381" y1="0" x2="-0.381" y2="60.96" width="0.1524" layer="16"/>
+</signal>
 </signals>
